Commit message: fix model + test position control

File: motoman/motoman_dual.urdf (robot description, URDF)
Before this commit: robot sda10f, 34 links, 33 joints
Links:
- link arm_left_link_1_s: geometry collision mesh filename=motoman_axis_s.stl; visual mesh filename=motoman_axis_s_v.stl
- link arm_left_link_2_l: geometry collision mesh filename=motoman_axis_l.stl; visual mesh filename=motoman_axis_l_v.stl
- link arm_left_link_3_e: geometry collision mesh filename=motoman_axis_e.stl; visual mesh filename=motoman_axis_e_v.stl
- link arm_left_link_4_u: geometry collision mesh filename=motoman_axis_u.stl; visual mesh filename=motoman_axis_u_v.stl
- link arm_left_link_5_r: geometry collision mesh filename=motoman_axis_r.stl; visual mesh filename=motoman_axis_r_v.stl
- link arm_left_link_6_b: geometry collision mesh filename=motoman_axis_b_remeshed.stl; visual mesh filename=motoman_axis_b_v.stl
- link arm_left_link_7_t: geometry collision mesh filename=motoman_axis_t.stl; visual mesh filename=motoman_axis_t_v.stl
- link arm_right_link_1_s: geometry collision mesh filename=motoman_axis_s.stl; visual mesh filename=motoman_axis_s_v.stl
- link arm_right_link_2_l: geometry collision mesh filename=motoman_axis_l.stl; visual mesh filename=motoman_axis_l_v.stl
- link arm_right_link_3_e: geometry collision mesh filename=motoman_axis_e.stl; visual mesh filename=motoman_axis_e_v.stl
- link arm_right_link_4_u: geometry collision mesh filename=motoman_axis_u.stl; visual mesh filename=motoman_axis_u_v.stl
- link arm_right_link_5_r: geometry collision mesh filename=motoman_axis_r.stl; visual mesh filename=motoman_axis_r_v.stl
- link arm_right_link_6_b: geometry collision mesh filename=motoman_axis_b_remeshed.stl; visual mesh filename=motoman_axis_b_v.stl
- link arm_right_link_7_t: geometry collision mesh filename=motoman_axis_t.stl; visual mesh filename=motoman_axis_t_v.stl
- link base_link: geometry collision mesh filename=motoman_base.stl; visual mesh filename=motoman_base_v.stl
- link left_inner_finger: geometry collision mesh filename=robotiq_arg2f_85_inner_finger.stl scale=0.001 0.001 0.001; visual mesh filename=robotiq_arg2f_85_inner_finger_v.stl scale=0.001 0.001 0.001
- link left_inner_knuckle: geometry collision mesh filename=robotiq_arg2f_85_inner_knuckle.stl scale=0.001 0.001 0.001; visual mesh filename=robotiq_arg2f_85_inner_knuckle_v.stl scale=0.001 0.001 0.001
- link left_outer_finger: geometry collision mesh filename=robotiq_arg2f_85_outer_finger.stl scale=0.001 0.001 0.001; visual mesh filename=robotiq_arg2f_85_outer_finger_v.stl scale=0.001 0.001 0.001
- link left_outer_knuckle: geometry collision mesh filename=robotiq_arg2f_85_outer_knuckle.stl scale=0.001 0.001 0.001; visual mesh filename=robotiq_arg2f_85_outer_knuckle_v.stl scale=0.001 0.001 0.001
- link onrobot_vgc10_base_link: mass 0.6 -> 0.00081386; geometry collision mesh filename=base_link.stl; visual mesh filename=base_link_v.stl
- link onrobot_vgc10_suction: mass 0.2 -> 0.00005331; geometry collision mesh filename=suction_cup.stl; visual mesh filename=suction_cup_v.stl
- link right_inner_finger: geometry collision mesh filename=robotiq_arg2f_85_inner_finger.stl scale=0.001 0.001 0.001; visual mesh filename=robotiq_arg2f_85_inner_finger_v.stl scale=0.001 0.001 0.001
- link right_inner_knuckle: geometry collision mesh filename=robotiq_arg2f_85_inner_knuckle.stl scale=0.001 0.001 0.001; visual mesh filename=robotiq_arg2f_85_inner_knuckle_v.stl scale=0.001 0.001 0.001
- link right_outer_finger: geometry collision mesh filename=robotiq_arg2f_85_outer_finger.stl scale=0.001 0.001 0.001; visual mesh filename=robotiq_arg2f_85_outer_finger_v.stl scale=0.001 0.001 0.001
- link right_outer_knuckle: geometry collision mesh filename=robotiq_arg2f_85_outer_knuckle.stl scale=0.001 0.001 0.001; visual mesh filename=robotiq_arg2f_85_outer_knuckle_v.stl scale=0.001 0.001 0.001
- link robotiq_arg2f_base_link: geometry collision mesh filename=robotiq_arg2f_base_link.stl; visual mesh filename=robotiq_arg2f_85_base_link_v.stl scale=0.001 0.001 0.001
- link torso_link_b1: geometry collision mesh filename=motoman_axis_b1_remeshed.stl; visual mesh filename=motoman_axis_b1_v.stl

Commit message: motion plan with ik

File: motoman/motoman_dual.urdf (robot description, URDF)
Before this commit: robot sda10f, 34 links, 33 joints
Joints:
- joint motoman_left_joint_ee: origin xyz=0 0 0.18 rpy=0 0 0 -> xyz=0 0 0.21 rpy=0 0 0
- joint motoman_right_joint_ee: origin xyz=0 0 0.135 rpy=0 0 0 -> xyz=0 0 0.18 rpy=0 0 0

Commit message: revert urdf offsets

File: motoman/motoman_dual.urdf (robot description, URDF)
Before this commit: robot sda10f, 34 links, 33 joints
Joints:
- joint motoman_left_joint_ee: origin xyz=0 0 0.21 rpy=0 0 0 -> xyz=0 0 0.18 rpy=0 0 0
- joint motoman_right_joint_ee: origin xyz=0 0 0.18 rpy=0 0 0 -> xyz=0 0 0.135 rpy=0 0 0
